Commit message: lidar and camera frames undetermine

File: csie-retriever_description/robots/pioneer3dx.xacro (robot description, xacro)
@@ -4,7 +4,8 @@
   <xacro:include filename="$(find csie-retriever_description)/urdf/sensors/hokuyo_utm30lx.urdf.xacro"/>
   <xacro:include filename="$(find csie-retriever_description)/urdf/sensors/_d435.urdf.xacro"/>
-  <sensor_d435 parent="base_link">
+  <!--xacro:include filename="$(find csie-retriever_description)/gazebo/gazebo.urdf.xacro"/-->
+<!--  <sensor_d435 parent="base_link">
     <origin xyz="0.110 0.0 0.3" rpy="0 0 0"/>
-  </sensor_d435>
+  </sensor_d435>-->
   <hokuyo_utm30lx parent="base_link" name="laser">
     <origin xyz="0.02 0 0.4" rpy="0 0 0"/>

File: csie-retriever_description/urdf/base/pioneer3dx_body.xacro (robot description, xacro)
@@ -1,5 +1,18 @@
 <?xml version="1.0"?>
 <robot xmlns:xacro="http://ros.org/wiki/xacro">
-  <xacro:include filename="$(find p2os_urdf)/defs/pioneer3dx_wheel.xacro"/>
+  <xacro:include filename="$(find csie-retriever_description)/urdf/base/pioneer3dx_wheel.xacro"/>
+    <link name="base_footprint">
+        <visual>
+          <origin xyz="0 0 0" rpy="0 0 0" />
+          <geometry>
+            <box size="0.001 0.001 0.001" />
+          </geometry>
+        </visual>
+     </link>
+     <joint name="base_footprint_joint" type="fixed">
+        <origin xyz="0 0 0" rpy="0 0 0" />
+        <child link="base_link" />
+        <parent link="base_footprint"/>
+    </joint>
   <!-- Chassis description -->
   <link name="base_link">
@@ -208,4 +221,6 @@
     <!-- Robot locomotion plugin -->
 	<plugin name="differential_drive_controller" filename="libgazebo_ros_diff_drive.so">
+<!--      <robotNamespace>/retriever</robotNamespace>-->
+      <robotNamespace>/</robotNamespace>
       <legacyMode>false</legacyMode>
       <alwaysOn>true</alwaysOn>
@@ -217,10 +232,9 @@
 	  <wheelTorque>5</wheelTorque>
       <wheelAcceleration>0</wheelAcceleration>
-      <robotNamespace>pioneer</robotNamespace>
 	  <commandTopic>cmd_vel</commandTopic>
 	  <odometryTopic>odom</odometryTopic>
       <odometrySource>ENCODER</odometrySource><!--Other option is World-->
 	  <odometryFrame>odom</odometryFrame>
-      <robotBaseFrame>base_link</robotBaseFrame>
+      <robotBaseFrame>base_footprint</robotBaseFrame>
       <publishTf>1</publishTf>
       <publishWheelTF>false</publishWheelTF>

Commit message: update navigation

File: csie-retriever_description/robots/pioneer3dx.xacro (robot description, xacro)
@@ -11,3 +11,6 @@
     <origin xyz="0.02 0 0.4" rpy="0 0 0"/>
   </hokuyo_utm30lx>
+  <hokuyo_utm30lx_back parent="base_link" name="laser_back">
+    <origin xyz="-0.1 0 0.4" rpy="0 0 ${pi}"/>
+  </hokuyo_utm30lx_back>
 </robot>

File: csie-retriever_description/urdf/sensors/hokuyo_utm30lx.urdf.xacro (robot description, xacro)
@@ -1,9 +1,8 @@
 <?xml version="1.0"?>
-<robot name="hokuyo_utm30lx" xmlns:xacro="http://ros.org/wiki/xacro">
+<robot xmlns:xacro="http://ros.org/wiki/xacro">
   <xacro:include filename="$(find csie-retriever_description)/urdf/sensors/hokuyo_utm30lx.gazebo.xacro" />
   <xacro:macro name="hokuyo_utm30lx" params="name parent *origin">
     <joint name="${name}_joint" type="fixed">
-      <!--origin xyz="0.105 0.000 0.229" rpy="0 0 0" /-->
-      <xacro:insert_block name="origin" />
+       <xacro:insert_block name="origin" />
       <!--<origin xyz="0.130 0.006 0.229" rpy="0 0 0" />-->
       <parent link="${parent}"/>
@@ -32,8 +31,7 @@
     <xacro:hokuyo_utm30lx_gazebo name="${name}" ros_topic="/scan" update_rate="40" ray_count="720" min_angle="-2" max_angle="2"/>
   </xacro:macro>
-  <xacro:macro name="hokuyo_utm30lx_back" params="name parent">
+  <xacro:macro name="hokuyo_utm30lx_back" params="name parent *origin">
     <joint name="${name}_joint" type="fixed">
-      <!--origin xyz="0.105 0.000 0.229" rpy="0 0 0" /-->
-      <origin xyz="-0.180 0.006 0.229" rpy="0 0 3.1415926535897931" />
+      <xacro:insert_block name="origin" />
       <parent link="${parent}"/>
       <child link="${name}_link"/>

Commit message: update

File: csie-retriever_description/robots/pioneer3dx.xacro (robot description, xacro)
@@ -5,12 +5,12 @@
   <xacro:include filename="$(find csie-retriever_description)/urdf/sensors/_d435.urdf.xacro"/>
   <!--xacro:include filename="$(find csie-retriever_description)/gazebo/gazebo.urdf.xacro"/-->
-<!--  <sensor_d435 parent="base_link">
+  <sensor_d435 parent="base_link">
     <origin xyz="0.110 0.0 0.3" rpy="0 0 0"/>
-  </sensor_d435>-->
+  </sensor_d435>
   <hokuyo_utm30lx parent="base_link" name="laser">
-    <origin xyz="0.02 0 0.4" rpy="0 0 0"/>
+    <origin xyz="0.1 0 0.3" rpy="0 0 0"/>
   </hokuyo_utm30lx>
   <hokuyo_utm30lx_back parent="base_link" name="laser_back">
-    <origin xyz="-0.1 0 0.4" rpy="0 0 ${pi}"/>
+    <origin xyz="-0.1 0 0.3" rpy="0 0 ${pi}"/>
   </hokuyo_utm30lx_back>
 </robot>

File: csie-retriever_description/urdf/sensors/_d435.urdf.xacro (robot description, xacro)
@@ -67,5 +67,5 @@
         <update_rate>20</update_rate>
         <camera>
-          <horizontal_fov>1.047198</horizontal_fov>
+          <horizontal_fov>1.347198</horizontal_fov>
           <image>
             <width>640</width>
@@ -75,5 +75,5 @@
           <clip>
             <near>0.05</near>
-            <far>3</far>
+            <far>8</far>
           </clip>
         </camera>
@@ -88,5 +88,8 @@
     <link name="camera_depth_frame"/>
     <joint name="camera_depth_optical_joint" type="fixed">
-      <origin xyz="0 0 0" rpy="${-M_PI/2} 0 ${-M_PI/2}" />
+      <!--original setting-->
+      <!--<origin xyz="0 0 0" rpy="${-M_PI/2} 0 ${-M_PI/2}" />-->
+      <!--modified for retiever-->
+      <origin xyz="0 0 0" rpy="${-M_PI/2} 0 0"/>
       <parent link="camera_depth_frame" />
       <child link="camera_depth_optical_frame" />
